File: hardware/cnc_1_0_0.brd (EAGLE design)
At the start: 78 x 126 mm, 88 parts, among them IC1 7805DT, IC2 4504D, IC3 4504D, IC4 4504D, IC5 7810, IC6 IL1212S, IC7 74AC244DW, Q2 25MHz, U2 ENC28J60-SSOP, X2 MSTBA2, X3 MSTBA2, X4 MSTBA2, X5 MSTBA2

Commit message: Updated to new version. Still in development.
Parts:
- removed R76, R77: 1k, rcl:R0805
- added C35, C37: 100nF, rcl:C0805K
- added C36, C38, C39: 1uF, rcl:C0805K
- added C40, C41: 10uF, rcl:C0805K
- added D1, D2: BAV103, diode:MINIMELF
- added IC8: OPA344N-SOT23, linear:SOT23-5
- added IC9: TR10, cnc:TR10
- added K1, K2: G2R2, relay:G2R2
- added L2: 22uH, inductors:DR127
- added Q4, Q5: BCW33SMD, transistor-npn:SOT23-BEC
- added Q7: BSS84, transistor-small-signal:SOT23
- added R17, R18, R20, R24, R25: 1k, rcl:R0805
- added R19: 0, rcl:R0805
- added R21, R22: 100k, rcl:R0805
- added R23: 1M, rcl:R0805
- added SJ4, SJ5: (no value), jumper:SJ
- added X6, X7: MSTBA2, con-phoenix-508:MSTBA2
- C28, C29, C30, C31, C32: value 100n -> 100nF
- C8: value 1uF -> 100nF
- moved C8 36.4 mm to (42.2, 31.0), turned to 0 degrees
- moved C7 35.5 mm to (44.4, 39.7), turned to 0 degrees
- moved JP39 34.4 mm to (8.82, 73.8)
- moved R15 30.6 mm to (8.54, 66.2), turned to 90 degrees
- moved JP3 29.3 mm to (8.13, 43.2), turned to 90 degrees
- moved R6 29.0 mm to (20.6, 73.8)
- moved X5 29.0 mm to (-1.00, 43.0)
- moved X4 29.0 mm to (-1.00, 56.0)
- moved X3 29.0 mm to (-1.00, 69.0)
- moved C6 29.0 mm to (62.0, 140.1)
- moved C4 29.0 mm to (59.6, 140.1)
- moved C5 29.0 mm to (57.0, 140.1)
- moved JP1 29.0 mm to (54.9, 131.6)
- moved X2 29.0 mm to (-1.91, 137.6)
- moved C27 29.0 mm to (31.4, 64.2)
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Connections:
- removed net N$45: C8.1, JP39.1, R77.2, X3.1
- removed net N$47: IC4.2, R76.1
- removed net RB17: SV1.7
- new net MIST_AIR: R25.1, SJ4.1
- new net MIST_OIL: R24.1, SJ5.1
- new net N$14: K2.S1, K2.S2, X7.1
- new net N$15: C7.1, IC8.3, R17.1
- new net N$16: IC8.4, R19.2, R20.1
- new net N$17: K2.O1, K2.O2
- new net N$18: K2.P1, K2.P2, X7.2
- new net N$19: K1.P1, K1.P2, X6.2
- new net N$20: K1.O1, K1.O2
- new net N$21: K1.S1, K1.S2, X6.1
- new net N$22: D2.A, K1.2, Q5.C
- new net N$23: D1.A, K2.2, Q4.C
- new net N$24: L1.2, Q7.3
- new net N$25: Q7.1, R23.2
- new net N$26: C40.1, IC9.P$1, L2.2
- new net N$27: Q4.B, R22.2, R24.2
- new net N$28: Q5.B, R21.2, R25.2
- new net RB14: SJ4.2, SV1.7
- new net RD1_10V: IC4.2, R18.2
- new net SPINDLE_ANALOG: C36.2, IC8.1, JP39.1, R19.1, X3.1
- net +10V: now also C35.1, IC8.5
- net +12V: now also C37.1, C38.1, C39.1, C41.1, C8.1, D1.C, D2.C, K1.1, K2.1, L2.1, Q7.2; no longer L1.2
- net +5V: now also IC9.P$3
- net GND: now also C35.2, C37.2, C38.2, C39.2, C40.2, C41.2, IC8.2, IC9.P$2, Q4.E, Q5.E, R20.2, R21.1, R22.1, R23.1
- net N$3: now also C36.1, R17.2, R18.1; no longer C7.1, R76.2, R77.1
- net RB12: now also SJ5.2
Routing:
- net +12V: track 133.0 -> 448.0 mm, vias 1 -> 2
- net MIST_OIL: track 0.00 -> 100.2 mm, vias 0 -> 2
- net SPINDLE_ANALOG: track 0.00 -> 91.8 mm, vias 0 -> 7
- net MIST_AIR: track 0.00 -> 86.5 mm, vias 0 -> 2
- net N$47: track 43.2 -> 0.00 mm, vias 2 -> 0
- net N$8: track 2.62 -> 31.0 mm, vias 0 -> 1
- net N$19: track 0.00 -> 22.0 mm
- net N$18: track 0.00 -> 21.9 mm
- net +10V: track 197.5 -> 219.0 mm
- net RD1_10V: track 0.00 -> 18.5 mm, vias 0 -> 2
- net RB14: track 0.00 -> 17.7 mm
- net RB12: track 0.00 -> 17.4 mm
- net N$3: track 4.95 -> 19.3 mm
- net N$26: track 0.00 -> 14.3 mm
- net N$21: track 0.00 -> 12.8 mm
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Other:
- board size 78 x 126 mm -> 78 x 155 mm
- board text added: "CNC_1_0_5"
- board text removed: "CNC_1_0_2"
