File: hardware/cnc_1_0_0.sch (EAGLE design)
At the start: 88 parts, among them IC1 7805DT, IC2 4504D, IC3 4504D, IC4 4504D, IC5 7810, IC6 IL1212S, IC7 74AC244DW, Q2 25MHz, U2 ENC28J60-SSOP, X2 MSTBA2, X3 MSTBA2, X4 MSTBA2, X5 MSTBA2

Commit message: Updated to new version. Still in development.
Parts:
- removed R76, R77: 1k, rcl:R-EU_R0805
- added C35, C37: 100nF, rcl:C-EUC0805K
- added C36, C38, C39: 1uF, rcl:C-EUC0805K
- added C40, C41: 10uF, rcl:C-EUC0805K
- added D1, D2: BAV103, diode:DIODE-MINIMELF
- added IC8: OPA344N-SOT23, linear:OPA344N-SOT23
- added IC9: TR10, cnc:TR10
- added K1, K2: G2R2, relay:G2R2
- added L2: 22uH, inductors:DR127
- added Q4, Q5: BCW33SMD, transistor-npn:BCW33SMD
- added Q7: BSS84, transistor-small-signal:BSS84
- added R17, R18, R20, R24, R25: 1k, rcl:R-EU_R0805
- added R19: 0, rcl:R-EU_R0805
- added R21, R22: 100k, rcl:R-EU_R0805
- added R23: 1M, rcl:R-EU_R0805
- added SJ4, SJ5: (no value), jumper:SJ
- added X6, X7: MSTBA2, con-phoenix-508:MSTBA2
- C28, C29, C30, C31, C32: value 100n -> 100nF
- C8: value 1uF -> 100nF
Connections:
- removed net N$45: C8.1, JP39.1, R77.2, X3-1.1
- removed net N$47: IC4A.AO, R76.1
- removed net RB17: SV1.7
- new net MIST_AIR: R25.1, SJ4.1
- new net MIST_OIL: R24.1, SJ5.1
- new net N$14: K22.S, K23.S, X7-1.1
- new net N$15: C7.1, IC8.+IN, R17.1
- new net N$16: IC8.-IN, R19.2, R20.1
- new net N$17: K22.O, K23.O
- new net N$18: K22.P, K23.P, X7-2.1
- new net N$19: K12.P, K13.P, X6-2.1
- new net N$20: K12.O, K13.O
- new net N$21: K12.S, K13.S, X6-1.1
- new net N$22: D2.A, K11.2, Q5.C
- new net N$23: D1.A, K21.2, Q4.C
- new net N$24: L1.2, Q7.D
- new net N$25: Q7.G, R23.2
- new net N$26: C40.1, IC9.IN, L2.2
- new net N$27: Q4.B, R22.2, R24.2
- new net N$28: Q5.B, R21.2, R25.2
- new net RB14: SJ4.2, SV1.7
- new net RD1_10V: IC4A.AO, R18.2
- new net SPINDLE_ANALOG: C36.2, IC8.OUT, JP39.1, R19.1, X3-1.1
- net +10V: now also C35.1, IC8.V+
- net +12V: now also C37.1, C38.1, C39.1, C41.1, C8.1, D1.C, D2.C, K11.1, K21.1, L2.1, Q7.S; no longer L1.2
- net +5V: now also IC9.OUT
- net GND: now also C35.2, C37.2, C38.2, C39.2, C40.2, C41.2, IC8.V-, IC9.GND, Q4.E, Q5.E, R20.2, R21.1, R22.1, R23.1
- net N$3: now also C36.1, R17.2, R18.1; no longer C7.1, R76.2, R77.1
- net RB12: now also SJ5.2
Other:
- note added: "Mist Air/Oil"
